File: _autosave-Brushless ESC.kicad_sch (KiCad schematic)
At the start: 40 parts, among them Q1 Q_NMOS_SGD, Q2 Q_NMOS_SGD, Q3 Q_NMOS_SGD, Q4 Q_NMOS_SGD, Q5 Q_NMOS_SGD, Q6 Q_NMOS_SGD, U2 STM32G491CET6

Commit message: i should probably back this up or something idk
Parts:
- added U3: TLV73333PDBV, Package_TO_SOT_SMD:SOT-23-5, symbol Regulator_Linear:TLV73333PDBV
Connections:
- net +3V3: now also U2.21 (VDDA), U2.24 (VDD), U2.36 (VDD), U2.48 (VDD), U3.5 (OUT)
- net GND: now also U2.19 (VSSA), U2.23 (VSS), U2.35 (VSS), U2.47 (VSS), U3.2 (GND)
- new net +BATT3V8: U3.1 (IN), U3.3 (EN)
- no-connect marks 0 -> 1
