File: Brushless ESC.kicad_sch (KiCad schematic)
At the start: 40 parts, among them Q1 Q_NMOS_SGD, Q2 Q_NMOS_SGD, Q3 Q_NMOS_SGD, Q4 Q_NMOS_SGD, Q5 Q_NMOS_SGD, Q6 Q_NMOS_SGD, U2 STM32G491CET6

Commit message: v1
Parts:
- added BT1: Battery, Connector_AMASS:AMASS_XT30U-F_1x02_P5.0mm_Vertical, symbol Device:Battery
- added C11, C12, C13, C14, C15: 100n, Capacitor_SMD:C_0402_1005Metric_Pad0.74x0.62mm_HandSolder, symbol Device:C_Small
- added C16: 1u, Capacitor_SMD:C_0402_1005Metric_Pad0.74x0.62mm_HandSolder, symbol Device:C_Small
- added C17: 10u, Capacitor_SMD:C_0402_1005Metric_Pad0.74x0.62mm_HandSolder, symbol Device:C_Small
- added C18: 100u, Capacitor_SMD:CP_Elec_10x10, symbol Device:C_Polarized
- added D7, D8: LED, Diode_SMD:D_0603_1608Metric_Pad1.05x0.95mm_HandSolder, symbol Device:LED
- added H1: U Phase Hole, Connector_Wire:SolderWire-2.5sqmm_1x01_D2.4mm_OD4.4mm, symbol Mechanical:MountingHole_Pad
- added H2: V Phase Hole, Connector_Wire:SolderWire-2.5sqmm_1x01_D2.4mm_OD4.4mm, symbol Mechanical:MountingHole_Pad
- added H3: W Phase Hole, Connector_Wire:SolderWire-2.5sqmm_1x01_D2.4mm_OD4.4mm, symbol Mechanical:MountingHole_Pad
- added J1: Conn_01x06, Connector_PinHeader_2.54mm:PinHeader_1x06_P2.54mm_Vertical, symbol Connector_Generic:Conn_01x06
- added J2, J3: Conn_01x03, Connector_PinHeader_2.54mm:PinHeader_1x03_P2.54mm_Vertical, symbol Connector_Generic:Conn_01x03
- added R10: 2k2_1%, Resistor_SMD:R_0402_1005Metric_Pad0.72x0.64mm_HandSolder, symbol Device:R
- added R11: 21k_1%, Resistor_SMD:R_0402_1005Metric_Pad0.72x0.64mm_HandSolder, symbol Device:R
- added R12: 1k_1%, Resistor_SMD:R_0402_1005Metric_Pad0.72x0.64mm_HandSolder, symbol Device:R
- added R13, R14: 43R, Resistor_SMD:R_0402_1005Metric_Pad0.72x0.64mm_HandSolder, symbol Device:R
- added TH1: NTCG103JF103, Resistor_SMD:R_0402_1005Metric_Pad0.72x0.64mm_HandSolder, symbol Device:Thermistor
- C7: footprint Capacitor_SMD:C_0805_2012Metric_Pad1.18x1.45mm_HandSolder -> Capacitor_SMD:C_0402_1005Metric_Pad0.74x0.62mm_HandSolder
- NT1, NT2, NT3, NT4, NT5, NT6: footprint (none) -> NetTie:NetTie-2_SMD_Pad0.5mm
- NT7: footprint (none) -> NetTie:NetTie-2_THT_Pad0.3mm
- Q1, Q2, Q3, Q4, Q5, Q6: footprint (none) -> Brushless ESC:2-5Q1S
- U1: footprint (none) -> Package_QFP:TQFP-48-1EP_7x7mm_P0.5mm_EP5x5mm
Connections:
- net SDI is gone; now on net MOSI: U1.15 (SDI)
- net SDO is gone; now on net MISO: U1.16 (SDO)
- net +3V3: now also U2.20 (VREF+), U2.21 (VDDA), U2.24 (VDD), U2.36 (VDD), U2.48 (VDD), C12.1, C13.1, C14.1, C15.1, C16.1, C17.1, J1.1 (Pin_1), J3.1 (Pin_1), R10.1, R14.2
- net +BATT: now also BT1.1 (+), C18.1, R11.1
- net -BATT: now also C7.2, U1.24 (CLK_IN), BT1.2 (-), C18.2, R12.2
- net CS: now also U2.12 (PA4)
- net Enable: now also U2.17 (PB1)
- net Fault: now also U2.16 (PB0)
- net GND: now also U2.19 (VSSA), U2.23 (VSS), U2.35 (VSS), U2.47 (VSS), C11.2, C12.2, C13.2, C14.2, C15.2, C16.2, C17.2, D7.1 (K), D8.1 (K), J1.3 (Pin_3), J2.3 (Pin_3), J3.3 (Pin_3), TH1.2; no longer C7.2, U1.24 (CLK_IN)
- net SCK: now also U2.13 (PA5)
- net U Cur: now also U2.8 (PA0)
- net U Out: now also H1.1
- net U Phase: now also C1.2
- net UH: now also U2.30 (PA8)
- net UL: now also U2.33 (PA11)
- net V Cur: now also U2.9 (PA1)
- net V Out: now also H2.1
- net V Phase: now also C2.2
- net VH: now also U2.31 (PA9)
- net VL: now also U2.34 (PA12)
- net W Cur: now also U2.10 (PA2)
- net W Out: now also H3.1
- net W Phase: now also C3.2
- net WH: now also U2.32 (PA10)
- net WL: now also U2.39 (PA15)
- net VBat: now reaches U2.11 (PA3)
- net VBat: now also R11.2, R12.1
- net MISO: now reaches U2.14 (PA6)
- net MOSI: now reaches U2.15 (PA7)
- net Temp: now reaches U2.18 (PB2)
- net Temp: now also R10.2, TH1.1
- net at U2.22 (PB10): now also R13.2
- net SWDIO: now reaches U2.37 (PA13)
- net SWDIO: now also J1.4 (Pin_4)
- net SWCLK: now reaches U2.38 (PA14)
- net SWCLK: now also J1.2 (Pin_2)
- net SWO: now reaches U2.40 (PB3)
- net SWO: now also J1.6 (Pin_6)
- net TX: now reaches U2.43 (PB6)
- net TX: now also J2.2 (Pin_2)
- net RX: now reaches U2.44 (PB7)
- net RX: now also J2.1 (Pin_1)
- net BOOT: now reaches U2.45 (PB8)
- net BOOT: now also J3.2 (Pin_2)
- net NRST: now reaches U2.7 (PG10)
- net NRST: now also C11.1, J1.5 (Pin_5)
- net U renamed U Sense-
- net U Sense-: no longer C1.2
- net U Sense renamed U Sense+
- net V renamed V Sense-
- net V Sense-: no longer C2.2
- net V Sense renamed V Sense+
- net V Sense+: no longer NT6.1
- net W renamed W Sense-
- net W Sense-: no longer C3.2
- net W Sense renamed W Sense+
- net W Sense+: now also NT6.1
- new net: D8.2 (A), R14.1
- new net: D7.2 (A), R13.1
- no-connect marks 0 -> 1
